File: hardware/rotary.kicad_sch (KiCad schematic)
At the start: 4 parts

Commit message: kinda works?
Parts:
- removed D?: D_Small, symbol Device:D_Small
Connections:
- net INT: now also U?.1 (~{RESET}/PB5)
Changed lines of the file:
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@@
 (kicad_sch (version 20211123) (generator eeschema)
   (paper "A4")
-  (junction (at 86.36 58.42) (diameter 0) (color 0 0 0 0)
-  )
   (junction (at 88.9 81.28) (diameter 0) (color 0 0 0 0)
   )
@@
   )
   (wire (pts (xy 116.84 81.28) (xy 96.52 81.28))
-    (stroke (width 0) (type default) (color 0 0 0 0))
-  )
-  (wire (pts (xy 86.36 43.18) (xy 86.36 48.26))
     (stroke (width 0) (type default) (color 0 0 0 0))
   )
@@
   )
   (wire (pts (xy 91.44 68.58) (xy 91.44 66.04))
-    (stroke (width 0) (type default) (color 0 0 0 0))
-  )
-  (wire (pts (xy 78.74 58.42) (xy 86.36 58.42))
     (stroke (width 0) (type default) (color 0 0 0 0))
   )
@@
     (stroke (width 0) (type default) (color 0 0 0 0))
   )
-  (wire (pts (xy 86.36 53.34) (xy 86.36 58.42))
-    (stroke (width 0) (type default) (color 0 0 0 0))
-  )
   (wire (pts (xy 63.5 35.56) (xy 109.22 35.56))
     (stroke (width 0) (type default) (color 0 0 0 0))
@@
     (stroke (width 0) (type default) (color 0 0 0 0))
   )
+  (wire (pts (xy 86.36 43.18) (xy 86.36 68.58))
+    (stroke (width 0) (type default) (color 0 0 0 0))
+  )
   (wire (pts (xy 86.36 43.18) (xy 109.22 43.18))
     (stroke (width 0) (type default) (color 0 0 0 0))
@@
     (stroke (width 0) (type default) (color 0 0 0 0))
   )
-  (wire (pts (xy 86.36 58.42) (xy 116.84 58.42))
+  (wire (pts (xy 78.74 58.42) (xy 116.84 58.42))
     (stroke (width 0) (type default) (color 0 0 0 0))
   )
@@
   )
   (wire (pts (xy 83.82 40.64) (xy 109.22 40.64))
+    (stroke (width 0) (type default) (color 0 0 0 0))
+  )
+  (wire (pts (xy 86.36 68.58) (xy 78.74 68.58))
     (stroke (width 0) (type default) (color 0 0 0 0))
   )
@@
     (pin "S2")
   )
-  (symbol (lib_id "Device:D_Small") (at 86.36 50.8 270) (unit 1)
-    (in_bom yes) (on_board yes)
-    (property "Reference" "D?" (id 0) (at 86.36 48.26 90)
-      (effects (font (size 1.27 1.27)) (justify left))
-    )
-    (property "Value" "D_Small" (id 1) (at 88.9 52.0699 90)
-      (effects (font (size 1.27 1.27)) (justify left) hide)
-    )
-    (property "Footprint" "" (id 2) (at 86.36 50.8 90)
-      (effects (font (size 1.27 1.27)) hide)
-    )
-    (property "Datasheet" "~" (id 3) (at 86.36 50.8 90)
-      (effects (font (size 1.27 1.27)) hide)
-    )
-    (pin "1")
-    (pin "2")
-  )
   (sheet_instances
     (path "/" (page "1"))
   )
   (symbol_instances
-    (path "/ac65d6cf-662e-44c7-a9ef-947c149c80cd"
-      (reference "D?") (unit 1) (value "D_Small") (footprint "")
-    )
     (path "/590d297e-44c5-40ef-85fc-cdbf70019459"
       (reference "J?") (unit 1) (value "Conn_01x05") (footprint "")
